File: envelope-generator/envelope-generator.kicad_sch (KiCad schematic)
At the start: 22 parts, among them SW1 Gate Button, SW2 AR/D Switch, SW3 AR/D Switch, U1 TL072

Commit message: Corrections to envelope generator
Parts:
- added D6: ~, symbol Device:D
- C1: value 10nF -> 47nF
- D4: value D -> ~
Connections:
- net at U1.6 (-), U1.7: now also D6.2 (A); no longer R8.2
- new net: D6.1 (K), R8.2
Other:
- moved on the sheet: D5, R8, R9
Changed lines of the file:
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@@
 	)
 	(junction
-		(at 240.03 76.2)
+		(at 232.41 105.41)
 		(diameter 0)
 		(color 0 0 0 0)
@@
 	(wire
 		(pts
-			(xy 250.19 76.2) (xy 254 76.2)
+			(xy 232.41 115.57) (xy 232.41 119.38)
 		)
 		(stroke
@@
 	(wire
 		(pts
-			(xy 240.03 76.2) (xy 242.57 76.2)
+			(xy 232.41 105.41) (xy 232.41 107.95)
 		)
 		(stroke
@@
 	(wire
 		(pts
+			(xy 232.41 88.9) (xy 232.41 95.25)
+		)
+		(stroke
+			(width 0)
+			(type default)
+		)
+	)
+	(wire
+		(pts
 			(xy 184.15 92.71) (xy 186.69 92.71)
 		)
@@
 	(wire
 		(pts
-			(xy 240.03 76.2) (xy 240.03 82.55)
+			(xy 232.41 105.41) (xy 243.84 105.41)
 		)
 		(stroke
@@
 	(wire
 		(pts
-			(xy 261.62 76.2) (xy 264.16 76.2)
+			(xy 232.41 127) (xy 232.41 129.54)
 		)
 		(stroke
@@
 	(wire
 		(pts
-			(xy 237.49 76.2) (xy 240.03 76.2)
+			(xy 232.41 102.87) (xy 232.41 105.41)
 		)
 		(stroke
@@
 	(wire
 		(pts
+			(xy 232.41 81.28) (xy 232.41 76.2)
+		)
+		(stroke
+			(width 0)
+			(type default)
+		)
+	)
+	(wire
+		(pts
 			(xy 144.78 57.15) (xy 147.32 57.15)
 		)
@@
 	(wire
 		(pts
-			(xy 226.06 76.2) (xy 229.87 76.2)
+			(xy 226.06 76.2) (xy 232.41 76.2)
 		)
 		(stroke
@@
 		)
 	)
+	(text_box "Diodes are signal diodes, such as 1N4148."
+		(exclude_from_sim no)
+		(at 30.48 44.45 0)
+		(size 20.32 7.62)
+		(stroke
+			(width 0)
+			(type default)
+		)
+		(fill
+			(type none)
+		)
+		(effects
+			(font
+				(size 1.27 1.27)
+			)
+			(justify left top)
+		)
+	)
 	(text "Attack"
 		(exclude_from_sim no)
@@
 				)
 				(justify left)
+				(hide yes)
 			)
 		)
@@
 	(symbol
 		(lib_id "power:GND")
-		(at 264.16 76.2 90)
+		(at 232.41 129.54 0)
 		(unit 1)
 		(exclude_from_sim no)
@@
 		(on_board yes)
 		(dnp no)
-		(fields_autoplaced yes)
 		(property "Reference" "#PWR011"
-			(at 270.51 76.2 0)
+			(at 232.41 135.89 0)
 			(effects
 				(font
@@
 		)
 		(property "Value" "GND"
-			(at 267.97 76.1999 90)
+			(at 234.442 134.366 0)
 			(effects
 				(font
@@
 		)
 		(property "Footprint" ""
-			(at 264.16 76.2 0)
+			(at 232.41 129.54 0)
 			(effects
 				(font
@@
 		)
 		(property "Datasheet" ""
-			(at 264.16 76.2 0)
+			(at 232.41 129.54 0)
 			(effects
 				(font
@@
 		)
 		(property "Description" "Power symbol creates a global label with name \"GND\" , ground"
-			(at 264.16 76.2 0)
+			(at 232.41 129.54 0)
 			(effects
 				(font
@@
 		(on_board yes)
 		(dnp no)
-		(fields_autoplaced yes)
 		(property "Reference" "D1"
-			(at 38.1 53.34 0)
+			(at 38.354 56.388 0)
 			(effects
 				(font
@@
 					(size 1.27 1.27)
 				)
+				(hide yes)
 			)
 		)
@@
 		(fields_autoplaced yes)
 		(property "Reference" "D4"
-			(at 167.64 81.2799 90)
+			(at 167.64 81.9149 90)
 			(effects
 				(font
@@
 			)
 		)
-		(property "Value" "D"
-			(at 167.64 83.8199 90)
+		(property "Value" "~"
+			(at 167.64 83.82 90)
 			(effects
 				(font
@@
 	(symbol
 		(lib_id "power:VAA")
-		(at 240.03 82.55 180)
+		(at 243.84 105.41 270)
 		(unit 1)
 		(exclude_from_sim no)
@@
 		(dnp no)
 		(property "Reference" "#PWR012"
-			(at 240.03 78.74 0)
+			(at 240.03 105.41 0)
 			(effects
 				(font
@@
 		)
 		(property "Value" "Output"
-			(at 240.03 87.122 0)
+			(at 250.698 105.41 90)
 			(effects
 				(font
@@
 		)
 		(property "Footprint" ""
-			(at 240.03 82.55 0)
+			(at 243.84 105.41 0)
 			(effects
 				(font
@@
 		)
 		(property "Datasheet" ""
-			(at 240.03 82.55 0)
+			(at 243.84 105.41 0)
 			(effects
 				(font
@@
 		)
 		(property "Description" "Power symbol creates a global label with name \"VAA\""
-			(at 240.03 82.55 0)
+			(at 243.84 105.41 0)
 			(effects
 				(font
@@
 	)
 	(symbol
+		(lib_id "Device:D")
+		(at 232.41 85.09 90)
+		(unit 1)
+		(exclude_from_sim no)
+		(in_bom yes)
+		(on_board yes)
+		(dnp no)
+		(fields_autoplaced yes)
+		(property "Reference" "D6"
+			(at 234.95 84.4549 90)
+			(effects
+				(font
+					(size 1.27 1.27)
+				)
+				(justify right)
+			)
+		)
+		(property "Value" "~"
+			(at 234.95 86.36 90)
+			(effects
+				(font
+					(size 1.27 1.27)
+				)
+				(justify right)
+			)
+		)
+		(property "Footprint" ""
+			(at 232.41 85.09 0)
+			(effects
+				(font
+					(size 1.27 1.27)
+				)
+				(hide yes)
+			)
+		)
+		(property "Datasheet" "~"
+			(at 232.41 85.09 0)
+			(effects
+				(font
+					(size 1.27 1.27)
+				)
+				(hide yes)
+			)
+		)
+		(property "Description" "Diode"
+			(at 232.41 85.09 0)
+			(effects
+				(font
+					(size 1.27 1.27)
+				)
+				(hide yes)
+			)
+		)
+		(property "Sim.Device" "D"
+			(at 232.41 85.09 0)
+			(effects
+				(font
+					(size 1.27 1.27)
+				)
+				(hide yes)
+			)
+		)
+		(property "Sim.Pins" "1=K 2=A"
+			(at 232.41 85.09 0)
+			(effects
+				(font
+					(size 1.27 1.27)
+				)
+				(hide yes)
+			)
+		)
+		(pin "2"
+		)
+		(pin "1"
+		)
+		(instances
+			(project "envelope-generator"
+				(path "/0cae5f57-7d92-4333-9827-99dd3c103f53"
+					(reference "D6")
+					(unit 1)
+				)
+			)
+		)
+	)
+	(symbol
 		(lib_id "Amplifier_Operational:TL072")
 		(at 33.02 39.37 90)
@@
 	(symbol
 		(lib_id "Device:R_US")
-		(at 233.68 76.2 270)
+		(at 232.41 99.06 180)
 		(unit 1)
 		(exclude_from_sim no)
@@
 		(on_board yes)
 		(dnp no)
-		(fields_autoplaced yes)
 		(property "Reference" "R8"
-			(at 233.68 69.85 90)
+			(at 235.966 97.79 0)
 			(effects
 				(font
@@
 		)
 		(property "Value" "1K"
-			(at 233.68 72.39 90)
+			(at 235.966 100.33 0)
 			(effects
 				(font
@@
 		)
 		(property "Footprint" ""
-			(at 233.426 77.216 90)
+			(at 231.394 98.806 90)
 			(effects
 				(font
@@
 		)
 		(property "Datasheet" "~"
-			(at 233.68 76.2 0)
+			(at 232.41 99.06 0)
 			(effects
 				(font
@@
 		)
 		(property "Description" "Resistor, US symbol"
-			(at 233.68 76.2 0)
+			(at 232.41 99.06 0)
 			(effects
 				(font
@@
 	(symbol
 		(lib_id "Device:LED")
-		(at 257.81 76.2 180)
+		(at 232.41 123.19 90)
 		(unit 1)
 		(exclude_from_sim no)
@@
 		(on_board yes)
 		(dnp no)
-		(fields_autoplaced yes)
 		(property "Reference" "D5"
-			(at 259.3975 68.58 0)
+			(at 236.728 124.46 90)
 			(effects
 				(font
@@
 		)
 		(property "Value" "LED"
-			(at 259.3975 71.12 0)
+			(at 236.728 121.92 90)
 			(effects
 				(font
@@
 		)
 		(property "Footprint" ""
-			(at 257.81 76.2 0)
+			(at 232.41 123.19 0)
 			(effects
 				(font
@@
 		)
 		(property "Datasheet" "~"
-			(at 257.81 76.2 0)
+			(at 232.41 123.19 0)
 			(effects
 				(font
@@
 		)
 		(property "Description" "Light emitting diode"
-			(at 257.81 76.2 0)
+			(at 232.41 123.19 0)
 			(effects
 				(font
@@
 	(symbol
 		(lib_id "Device:R_US")
-		(at 246.38 76.2 270)
+		(at 232.41 111.76 180)
 		(unit 1)
 		(exclude_from_sim no)
@@
 		(on_board yes)
 		(dnp no)
-		(fields_autoplaced yes)
 		(property "Reference" "R9"
-			(at 246.38 69.85 90)
+			(at 235.966 110.744 0)
 			(effects
 				(font
@@
 		)
 		(property "Value" "1K"
-			(at 246.38 72.39 90)
+			(at 235.966 113.284 0)
 			(effects
 				(font
@@
 		)
 		(property "Footprint" ""
-			(at 246.126 77.216 90)
+			(at 231.394 111.506 90)
 			(effects
 				(font
@@
 		)
 		(property "Datasheet" "~"
-			(at 246.38 76.2 0)
+			(at 232.41 111.76 0)
 			(effects
 				(font
@@
 		)
 		(property "Description" "Resistor, US symbol"
-			(at 246.38 76.2 0)
+			(at 232.41 111.76 0)
 			(effects
 				(font
@@
 			)
 		)
-		(property "Value" "10nF"
+		(property "Value" "47nF"
 			(at 77.47 64.77 90)
 			(effects
