File: envelope-generator/envelope-generator.kicad_sch (KiCad schematic)
At the start: 23 parts, among them SW1 Gate Button, SW2 AR/D Switch, SW3 AR/D Switch, U1 TL072

Commit message: Fix error in envolpe generator schematic
Parts:
- RV2: value 250K -> 1M
Changed lines of the file:
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@@
 			)
 		)
-		(property "Value" "250K"
+		(property "Value" "1M"
 			(at 180.34 99.06 90)
 			(effects
